Commit message: feat:add pedestal

File: iiwa_ur_description/urdf/iiwa7_ur5.urdf (robot description, URDF)
Before this commit: robot iiwa_ur5, 20 links, 19 joints
Links:
- added link iiwa_pedestal; collision mesh filename=package://iiwa_ur_description/meshes/pedestal.STL; visual mesh filename=package://iiwa_ur_description/meshes/pedestal.STL
- added link ur_pedestal; collision mesh filename=package://iiwa_ur_description/meshes/pedestal.STL; visual mesh filename=package://iiwa_ur_description/meshes/pedestal.STL
Joints:
- added joint iiwa_pedestal_to_world: type fixed, parent iiwa_link_0, child iiwa_pedestal, origin xyz=0 0 0 rpy=0 0 0.7854
- added joint ur_pedestal_to_world: type fixed, parent base_link, child ur_pedestal, origin xyz=0 0 0 rpy=0 0 0.7854
- joint world_iiwa_joint: origin xyz=0.0 0.0 0 rpy=0.0 0.0 0.0 -> xyz=0.0 0.0 0.7 rpy=0.0 0.0 0.0
- joint world_ur_joint: origin xyz=1.0 0.0 0 rpy=0.0 0.0 3.14159265359 -> xyz=1.2 0.0 0.7 rpy=0.0 0.0 3.14159265359

File: iiwa_ur_description/urdf/iiwa7_ur5.urdf.xacro (robot description, xacro)
@@ -5,4 +5,8 @@
   <material name="grey">
     <color rgba="0.5 0.5 0.5 1.0"/>
+  </material>
+  <!--black-->
+  <material name="black">
+    <color rgba="0.0 0.0 0.0  1.0"/>
   </material>
   <!--| iiwa |-->
@@ -28,12 +32,84 @@
   <!-- world_iiwa_joint -->
   <xacro:iiwa7 hardware_interface="$(arg hardware_interface)" robot_name="$(arg robot_name)" parent="world">
-    <origin xyz="0.0 0.0 0" rpy="0.0 0.0 0.0" />
+    <origin xyz="0.0 0.0 0.7" rpy="0.0 0.0 0.0" />
   </xacro:iiwa7>
   <!-- world_ur_joint -->
   <joint name="world_${prefix_ur}_joint" type="fixed">
     <parent link="world" />
-    <child link = "base_link" />
-    <origin xyz="1.0 0.0 0" rpy="0.0 0.0 ${PI}" />
+    <child link="base_link" />
+    <origin xyz="1.2 0.0 0.7" rpy="0.0 0.0 ${PI}" />
   </joint>
-  <!-- add optical table -->
+  <!-- add iiwa pedestal -->
+  <link name="${prefix_iiwa}_pedestal">
+    <visual>
+      <origin rpy="0 0 0" xyz="0 0 0"/>
+      <geometry>
+        <mesh filename="package://iiwa_ur_description/meshes/pedestal.STL"/>
+      </geometry>
+      <material name="grey"/>
+    </visual>
+    <collision>
+      <origin rpy="0 0 0" xyz="0 0 0"/>
+      <geometry>
+        <mesh filename="package://iiwa_ur_description/meshes/pedestal.STL"/>
+      </geometry>
+    </collision>
+  </link>
+  <!-- add ur pedestal -->
+  <link name="${prefix_ur}_pedestal">
+    <visual>
+      <origin rpy="0 0 0" xyz="0 0 0"/>
+      <geometry>
+        <mesh filename="package://iiwa_ur_description/meshes/pedestal.STL"/>
+      </geometry>
+      <material name="grey"/>
+    </visual>
+    <collision>
+      <origin rpy="0 0 0" xyz="0 0 0"/>
+      <geometry>
+        <mesh filename="package://iiwa_ur_description/meshes/pedestal.STL"/>
+      </geometry>
+    </collision>
+  </link>
+  <joint name="${prefix_iiwa}_pedestal_to_world" type="fixed">
+    <parent link="iiwa_link_0"/>
+    <child link="${prefix_iiwa}_pedestal"/>
+    <origin rpy="0 0 0.7854" xyz="0 0 0"/>
+  </joint>
+  <joint name="${prefix_ur}_pedestal_to_world" type="fixed">
+    <parent link="base_link"/>
+    <child link="${prefix_ur}_pedestal"/>
+    <origin rpy="0 0 0.7854" xyz="0 0 0"/>
+  </joint>
+  <!-- add optical table, not display well yet -->
+  <!-- world_iiwa_joint -->
+  <!--   <xacro:iiwa7 hardware_interface="$(arg hardware_interface)" robot_name="$(arg robot_name)" parent="world">
+    <origin xyz="0.0 0.0 0.858" rpy="0.0 0.0 0.0" />
+  </xacro:iiwa7> -->
+  <!-- world_ur_joint -->
+  <!--   <joint name="world_${prefix_ur}_joint" type="fixed">
+    <parent link="world" />
+    <child link="base_link" />
+    <origin xyz="1.0 0.0 0.858" rpy="0.0 0.0 ${PI}" />
+  </joint> -->
+  <!--   <link name="optical_table">
+    <visual>
+    <origin xyz="0.0 0.0 0" rpy="0.0 0.0 0.0" />
+      <geometry>
+        <mesh filename="package://iiwa_ur_description/meshes/optical_table.STL"/>
+      </geometry>
+      <material name="grey"/>
+    </visual>
+    <collision>
+    <origin xyz="0.0 0.0 0" rpy="0.0 0.0 0.0" />
+      <geometry>
+        <mesh filename="package://iiwa_ur_description/meshes/optical_table.STL"/>
+      </geometry>
+    </collision>
+  </link>
+  <joint name="iiwa_to_optical" type="fixed">
+    <parent link="iiwa_link_0"/>
+    <child link="optical_table"/>
+    <origin xyz="0.0 0.0 -0.788" rpy="${PI/2.0} 0 0.0" />
+  </joint> -->
 </robot>
