Commit message: feat: options to load pedestal whether or not

File: iiwa_ur_description/urdf/iiwa7_ur5.urdf.xacro (robot description, xacro)
@@ -32,5 +32,5 @@
   <!-- world_iiwa_joint -->
   <xacro:iiwa7 hardware_interface="$(arg hardware_interface)" robot_name="$(arg robot_name)" parent="world">
-    <origin xyz="0.0 0.0 0.7" rpy="0.0 0.0 0.0" />
+    <origin xyz="0.0 0.0 0.0" rpy="0.0 0.0 0.0" />
   </xacro:iiwa7>
   <!-- world_ur_joint -->
@@ -38,78 +38,5 @@
     <parent link="world" />
     <child link="base_link" />
-    <origin xyz="1.2 0.0 0.7" rpy="0.0 0.0 ${PI}" />
+    <origin xyz="1.2 0.0 0.0" rpy="0.0 0.0 ${PI}" />
   </joint>
-  <!-- add iiwa pedestal -->
-  <link name="${prefix_iiwa}_pedestal">
-    <visual>
-      <origin rpy="0 0 0" xyz="0 0 0"/>
-      <geometry>
-        <mesh filename="package://iiwa_ur_description/meshes/pedestal.STL"/>
-      </geometry>
-      <material name="grey"/>
-    </visual>
-    <collision>
-      <origin rpy="0 0 0" xyz="0 0 0"/>
-      <geometry>
-        <mesh filename="package://iiwa_ur_description/meshes/pedestal.STL"/>
-      </geometry>
-    </collision>
-  </link>
-  <!-- add ur pedestal -->
-  <link name="${prefix_ur}_pedestal">
-    <visual>
-      <origin rpy="0 0 0" xyz="0 0 0"/>
-      <geometry>
-        <mesh filename="package://iiwa_ur_description/meshes/pedestal.STL"/>
-      </geometry>
-      <material name="grey"/>
-    </visual>
-    <collision>
-      <origin rpy="0 0 0" xyz="0 0 0"/>
-      <geometry>
-        <mesh filename="package://iiwa_ur_description/meshes/pedestal.STL"/>
-      </geometry>
-    </collision>
-  </link>
-  <joint name="${prefix_iiwa}_pedestal_to_world" type="fixed">
-    <parent link="iiwa_link_0"/>
-    <child link="${prefix_iiwa}_pedestal"/>
-    <origin rpy="0 0 0.7854" xyz="0 0 0"/>
-  </joint>
-  <joint name="${prefix_ur}_pedestal_to_world" type="fixed">
-    <parent link="base_link"/>
-    <child link="${prefix_ur}_pedestal"/>
-    <origin rpy="0 0 0.7854" xyz="0 0 0"/>
-  </joint>
-  <!-- add optical table, not display well yet -->
-  <!-- world_iiwa_joint -->
-  <!--   <xacro:iiwa7 hardware_interface="$(arg hardware_interface)" robot_name="$(arg robot_name)" parent="world">
-    <origin xyz="0.0 0.0 0.858" rpy="0.0 0.0 0.0" />
-  </xacro:iiwa7> -->
-  <!-- world_ur_joint -->
-  <!--   <joint name="world_${prefix_ur}_joint" type="fixed">
-    <parent link="world" />
-    <child link="base_link" />
-    <origin xyz="1.0 0.0 0.858" rpy="0.0 0.0 ${PI}" />
-  </joint> -->
-  <!--   <link name="optical_table">
-    <visual>
-    <origin xyz="0.0 0.0 0" rpy="0.0 0.0 0.0" />
-      <geometry>
-        <mesh filename="package://iiwa_ur_description/meshes/optical_table.STL"/>
-      </geometry>
-      <material name="grey"/>
-    </visual>
-    <collision>
-    <origin xyz="0.0 0.0 0" rpy="0.0 0.0 0.0" />
-      <geometry>
-        <mesh filename="package://iiwa_ur_description/meshes/optical_table.STL"/>
-      </geometry>
-    </collision>
-  </link>
-  <joint name="iiwa_to_optical" type="fixed">
-    <parent link="iiwa_link_0"/>
-    <child link="optical_table"/>
-    <origin xyz="0.0 0.0 -0.788" rpy="${PI/2.0} 0 0.0" />
-  </joint> -->
 </robot>

File: iiwa_ur_description/urdf/iiwa7_ur5_joint_limited.urdf.xacro (robot description, xacro)
@@ -40,5 +40,5 @@
   <!-- world_iiwa_joint -->
   <xacro:iiwa7 hardware_interface="$(arg hardware_interface)" robot_name="$(arg robot_name)" parent="world">
-    <origin xyz="0.0 0.0 0.7" rpy="0.0 0.0 0.0" />
+    <origin xyz="0.0 0.0 0.0" rpy="0.0 0.0 0.0" />
   </xacro:iiwa7>
   <!-- world_ur_joint -->
@@ -46,78 +46,5 @@
     <parent link="world" />
     <child link="base_link" />
-    <origin xyz="1.2 0.0 0.7" rpy="0.0 0.0 ${PI}" />
+    <origin xyz="1.2 0.0 0.0" rpy="0.0 0.0 ${PI}" />
   </joint>
-  <!-- add iiwa pedestal -->
-  <link name="${prefix_iiwa}_pedestal">
-    <visual>
-      <origin rpy="0 0 0" xyz="0 0 0"/>
-      <geometry>
-        <mesh filename="package://iiwa_ur_description/meshes/pedestal.STL"/>
-      </geometry>
-      <material name="grey"/>
-    </visual>
-    <collision>
-      <origin rpy="0 0 0" xyz="0 0 0"/>
-      <geometry>
-        <mesh filename="package://iiwa_ur_description/meshes/pedestal.STL"/>
-      </geometry>
-    </collision>
-  </link>
-  <!-- add ur pedestal -->
-  <link name="${prefix_ur}_pedestal">
-    <visual>
-      <origin rpy="0 0 0" xyz="0 0 0"/>
-      <geometry>
-        <mesh filename="package://iiwa_ur_description/meshes/pedestal.STL"/>
-      </geometry>
-      <material name="grey"/>
-    </visual>
-    <collision>
-      <origin rpy="0 0 0" xyz="0 0 0"/>
-      <geometry>
-        <mesh filename="package://iiwa_ur_description/meshes/pedestal.STL"/>
-      </geometry>
-    </collision>
-  </link>
-  <joint name="${prefix_iiwa}_pedestal_to_world" type="fixed">
-    <parent link="iiwa_link_0"/>
-    <child link="${prefix_iiwa}_pedestal"/>
-    <origin rpy="0 0 0.7854" xyz="0 0 0"/>
-  </joint>
-  <joint name="${prefix_ur}_pedestal_to_world" type="fixed">
-    <parent link="base_link"/>
-    <child link="${prefix_ur}_pedestal"/>
-    <origin rpy="0 0 0.7854" xyz="0 0 0"/>
-  </joint>
-  <!-- add optical table, not display well yet -->
-  <!-- world_iiwa_joint -->
-  <!--   <xacro:iiwa7 hardware_interface="$(arg hardware_interface)" robot_name="$(arg robot_name)" parent="world">
-    <origin xyz="0.0 0.0 0.858" rpy="0.0 0.0 0.0" />
-  </xacro:iiwa7> -->
-  <!-- world_ur_joint -->
-  <!--   <joint name="world_${prefix_ur}_joint" type="fixed">
-    <parent link="world" />
-    <child link="base_link" />
-    <origin xyz="1.0 0.0 0.858" rpy="0.0 0.0 ${PI}" />
-  </joint> -->
-  <!--   <link name="optical_table">
-    <visual>
-    <origin xyz="0.0 0.0 0" rpy="0.0 0.0 0.0" />
-      <geometry>
-        <mesh filename="package://iiwa_ur_description/meshes/optical_table.STL"/>
-      </geometry>
-      <material name="grey"/>
-    </visual>
-    <collision>
-    <origin xyz="0.0 0.0 0" rpy="0.0 0.0 0.0" />
-      <geometry>
-        <mesh filename="package://iiwa_ur_description/meshes/optical_table.STL"/>
-      </geometry>
-    </collision>
-  </link>
-  <joint name="iiwa_to_optical" type="fixed">
-    <parent link="iiwa_link_0"/>
-    <child link="optical_table"/>
-    <origin xyz="0.0 0.0 -0.788" rpy="${PI/2.0} 0 0.0" />
-  </joint> -->
 </robot>

Commit message: add use_pedestal option

File: iiwa_ur_description/urdf/iiwa7_ur5.urdf.xacro (robot description, xacro)
@@ -10,7 +10,4 @@
     <color rgba="0.0 0.0 0.0  1.0"/>
   </material>
-  <!-- prefix of two arms -->
-  <xacro:property name="prefix_iiwa" value="$(arg robot_name)" />
-  <xacro:property name="prefix_ur" value="ur" />
   <!--| iiwa |-->
   <!-- Import Rviz colors -->
@@ -30,4 +27,7 @@
   <!-- ur5 -->
   <xacro:ur5_robot prefix="" joint_limited="false" transmission_hw_interface="$(arg transmission_hw_interface)" />
+  <!-- prefix of two arms -->
+  <xacro:property name="prefix_iiwa" value="$(arg robot_name)" />
+  <xacro:property name="prefix_ur" value="ur" />
   <link name="world" />
   <!-- world_iiwa_joint -->

File: iiwa_ur_description/urdf/iiwa7_ur5_joint_limited.urdf (robot description, URDF)
Before this commit: robot iiwa_ur, 20 links, 19 joints
Joints:
- joint shoulder_lift_joint: limit lower=-6.28318530718 upper=6.28318530718 effort=150.0 velocity=3.15 -> lower=-3.14159265359 upper=3.14159265359 effort=150.0 velocity=3.15
- joint shoulder_pan_joint: limit lower=-6.28318530718 upper=6.28318530718 effort=150.0 velocity=3.15 -> lower=-3.14159265359 upper=3.14159265359 effort=150.0 velocity=3.15
- joint wrist_1_joint: limit lower=-6.28318530718 upper=6.28318530718 effort=28.0 velocity=3.2 -> lower=-3.14159265359 upper=3.14159265359 effort=28.0 velocity=3.2
- joint wrist_2_joint: limit lower=-6.28318530718 upper=6.28318530718 effort=28.0 velocity=3.2 -> lower=-3.14159265359 upper=3.14159265359 effort=28.0 velocity=3.2
- joint wrist_3_joint: limit lower=-6.28318530718 upper=6.28318530718 effort=28.0 velocity=3.2 -> lower=-3.14159265359 upper=3.14159265359 effort=28.0 velocity=3.2

File: iiwa_ur_description/urdf/iiwa7_ur5_joint_limited.urdf.xacro (robot description, xacro)
@@ -10,7 +10,4 @@
     <color rgba="0.0 0.0 0.0  1.0"/>
   </material>
-  <!-- prefix of two arms -->
-  <xacro:property name="prefix_iiwa" value="$(arg robot_name)" />
-  <xacro:property name="prefix_ur" value="ur" />
   <!--| iiwa |-->
   <!-- Import Rviz colors -->
@@ -30,5 +27,7 @@
   <!-- ur5 -->
   <xacro:ur5_robot prefix="" joint_limited="true" shoulder_pan_lower_limit="${-pi}" shoulder_pan_upper_limit="${pi}" shoulder_lift_lower_limit="${-pi}" shoulder_lift_upper_limit="${pi}" elbow_joint_lower_limit="${-pi}" elbow_joint_upper_limit="${pi}" wrist_1_lower_limit="${-pi}" wrist_1_upper_limit="${pi}" wrist_2_lower_limit="${-pi}" wrist_2_upper_limit="${pi}" wrist_3_lower_limit="${-pi}" wrist_3_upper_limit="${pi}" transmission_hw_interface="$(arg transmission_hw_interface)" />
-  <link name="world" />
+  <!-- prefix of two arms -->
+  <xacro:property name="prefix_iiwa" value="$(arg robot_name)" />
+  <xacro:property name="prefix_ur" value="ur" /><link name="world" />
   <!-- world_iiwa_joint -->
   <xacro:iiwa7 hardware_interface="$(arg hardware_interface)" robot_name="$(arg robot_name)" robot_namespace="$(arg robot_namespace)" parent="world">

File: iiwa_ur_description/urdf/iiwa7_ur5_pedestal.urdf (robot description, URDF)
Before this commit: robot iiwa_ur, 20 links, 19 joints
Links:
- added link iiwa_pedestal; collision mesh filename=package://iiwa_ur_description/meshes/pedestal.STL; visual mesh filename=package://iiwa_ur_description/meshes/pedestal.STL
- added link ur_pedestal; collision mesh filename=package://iiwa_ur_description/meshes/pedestal.STL; visual mesh filename=package://iiwa_ur_description/meshes/pedestal.STL
Joints:
- added joint iiwa_pedestal_to_world: type fixed, parent iiwa_link_0, child iiwa_pedestal, origin xyz=0 0 0 rpy=0 0 0.7854
- added joint ur_pedestal_to_world: type fixed, parent base_link, child ur_pedestal, origin xyz=0 0 0 rpy=0 0 0.7854
- joint world_iiwa_joint: origin xyz=0.0 0.0 0.0 rpy=0.0 0.0 0.0 -> xyz=0.0 0.0 0.7 rpy=0.0 0.0 0.0
- joint world_ur_joint: origin xyz=1.2 0.0 0.0 rpy=0.0 0.0 3.14159265359 -> xyz=1.2 0.0 0.7 rpy=0.0 0.0 3.14159265359

File: iiwa_ur_description/urdf/iiwa7_ur5_pedestal.urdf.xacro (robot description, xacro)
@@ -10,7 +10,4 @@
     <color rgba="0.0 0.0 0.0  1.0"/>
   </material>
-  <!-- prefix of two arms -->
-  <xacro:property name="prefix_iiwa" value="$(arg robot_name)" />
-  <xacro:property name="prefix_ur" value="ur" />
   <!--| iiwa |-->
   <!-- Import Rviz colors -->
@@ -25,9 +22,12 @@
   <xacro:arg name="transmission_hw_interface" default="hardware_interface/PositionJointInterface"/>
   <!-- common stuff -->
-  <xacro:include filename="$(find ur_description)/urdf/common.gazebo.xacro" />
+  <!-- <xacro:include filename="$(find ur_description)/urdf/common.gazebo.xacro" /> -->
   <!-- ur5 -->
   <xacro:include filename="$(find ur_description)/urdf/ur5.urdf.xacro" />
   <!-- ur5 -->
   <xacro:ur5_robot prefix="" joint_limited="false" transmission_hw_interface="$(arg transmission_hw_interface)" />
+  <!-- prefix of two arms -->
+  <xacro:property name="prefix_iiwa" value="$(arg robot_name)" />
+  <xacro:property name="prefix_ur" value="ur" />
   <link name="world" />
   <!-- world_iiwa_joint -->

File: iiwa_ur_description/urdf/iiwa7_ur5_pedestal_joint_limited.urdf (robot description, URDF)
Before this commit: robot iiwa_ur, 20 links, 19 joints
Links:
- added link iiwa_pedestal; collision mesh filename=package://iiwa_ur_description/meshes/pedestal.STL; visual mesh filename=package://iiwa_ur_description/meshes/pedestal.STL
- added link ur_pedestal; collision mesh filename=package://iiwa_ur_description/meshes/pedestal.STL; visual mesh filename=package://iiwa_ur_description/meshes/pedestal.STL
Joints:
- added joint iiwa_pedestal_to_world: type fixed, parent iiwa_link_0, child iiwa_pedestal, origin xyz=0 0 0 rpy=0 0 0.7854
- added joint ur_pedestal_to_world: type fixed, parent base_link, child ur_pedestal, origin xyz=0 0 0 rpy=0 0 0.7854
- joint shoulder_lift_joint: limit lower=-6.28318530718 upper=6.28318530718 effort=150.0 velocity=3.15 -> lower=-3.14159265359 upper=3.14159265359 effort=150.0 velocity=3.15
- joint shoulder_pan_joint: limit lower=-6.28318530718 upper=6.28318530718 effort=150.0 velocity=3.15 -> lower=-3.14159265359 upper=3.14159265359 effort=150.0 velocity=3.15
- joint world_iiwa_joint: origin xyz=0.0 0.0 0.0 rpy=0.0 0.0 0.0 -> xyz=0.0 0.0 0.7 rpy=0.0 0.0 0.0
- joint world_ur_joint: origin xyz=1.2 0.0 0.0 rpy=0.0 0.0 3.14159265359 -> xyz=1.2 0.0 0.7 rpy=0.0 0.0 3.14159265359
- joint wrist_1_joint: limit lower=-6.28318530718 upper=6.28318530718 effort=28.0 velocity=3.2 -> lower=-3.14159265359 upper=3.14159265359 effort=28.0 velocity=3.2
- joint wrist_2_joint: limit lower=-6.28318530718 upper=6.28318530718 effort=28.0 velocity=3.2 -> lower=-3.14159265359 upper=3.14159265359 effort=28.0 velocity=3.2
- joint wrist_3_joint: limit lower=-6.28318530718 upper=6.28318530718 effort=28.0 velocity=3.2 -> lower=-3.14159265359 upper=3.14159265359 effort=28.0 velocity=3.2

File: iiwa_ur_description/urdf/iiwa7_ur5_pedestal_joint_limited.urdf.xacro (robot description, xacro)
@@ -10,7 +10,4 @@
     <color rgba="0.0 0.0 0.0  1.0"/>
   </material>
-  <!-- prefix of two arms -->
-  <xacro:property name="prefix_iiwa" value="$(arg robot_name)" />
-  <xacro:property name="prefix_ur" value="ur" />
   <!--| iiwa |-->
   <!-- Import Rviz colors -->
@@ -38,4 +35,7 @@
     transmission_hw_interface="$(arg transmission_hw_interface)"
   />
+  <!-- prefix of two arms -->
+  <xacro:property name="prefix_iiwa" value="$(arg robot_name)" />
+  <xacro:property name="prefix_ur" value="ur" />
   <link name="world" />
   <!-- world_iiwa_joint -->
